File: PEKG.kicad_sch (KiCad schematic)
At the start: 76 parts, among them J1 USB_C_Receptacle, J2 AudioJack3, U10 74LVC1G125, U11 74LVC1G125, U12 NCS21802DMR2G, U13 NCS21802DMR2G, U14 NCS21802DMR2G, U4 74LVC2G74, U5 TS5A63157DBV, U6 TS5A63157DBV, U7 TS5A63157DBV, U8 NCS21802DMR2G, U9 74LVC1G125

Commit message: Updates schematic, tests.
Fixed git issue
Parts:
- removed C1, C2, C26, C7: 100n, Capacitor_SMD:C_0603_1608Metric_Pad1.08x0.95mm_HandSolder, symbol Device:C
- removed C27: 1u, Capacitor_SMD:C_0603_1608Metric_Pad1.08x0.95mm_HandSolder, symbol Device:C
- added C28, C29: 10n, Capacitor_SMD:C_0603_1608Metric_Pad1.08x0.95mm_HandSolder, symbol Device:C
- added C30: 1u, Capacitor_SMD:C_0603_1608Metric_Pad1.08x0.95mm_HandSolder, symbol Device:C
- added JP1, JP3: Jumper_2_Bridged, Jumper:SolderJumper-2_P1.3mm_Bridged_RoundedPad1.0x1.5mm, symbol Jumper:Jumper_2_Bridged
- added JP2, JP4: Jumper_2_Open, Jumper:SolderJumper-2_P1.3mm_Open_RoundedPad1.0x1.5mm, symbol Jumper:Jumper_2_Open
- C5: value 1u -> 100n
- C9: value 100n -> 1u
- R12: value 100k -> inf -> 1k
- R25: value 190k -> 100k
- R4, R5, R6, R7: value 10k -> 1k
- R8, R9: value 10k -> 100k
Connections:
- net VCC is gone; now on net VBUS: C10.1, C3.1, C5.1, C6.1, C8.1, D1.2 (A), D2.2 (A), R18.2, R28.2, U12.8 (V+), U13.8 (V+), U14.8 (V+), U8.8 (V+)
- net VEE is gone; now on net GND: C10.2, C4.2, C5.2, C6.2, C9.2, D1.1 (K), D2.1 (K), U12.4 (V-), U13.4 (V-), U14.4 (V-), U8.4 (V-)
- net 2.5V: now also JP1.1 (A)
- net DC_COMPENSATION: now also C28.2, JP1.2 (B), JP2.2 (B); no longer C22.1, R16.1, U13.1
- net GND: now also C30.2; no longer C4.1, C9.1
- net VBUS: now also C4.1, C9.1, C30.1
- net at R7.1, R8.2, U12.2 (-): now also C29.1
- net at R6.1, R9.2, U12.3 (+): now also C28.1
- net GAIN_100_OUTPUT: no longer names the net of C24.1, R25.1, U14.1
- net GAIN_100_OUTPUT: now also JP4.1 (A); no longer R30.2
- net GAIN_5_OUTPUT renamed GAIN_500_OUTPUT
- net GAIN_500_OUTPUT: now also C29.2, JP3.1 (A)
- new net: C22.1, JP2.1 (A), R16.1, U13.1
- new net GAIN_5000_OUTPUT: JP3.2 (B), JP4.2 (B), R30.2
Other:
- note added: "DODAJ JUMPER KOJI ISKLJUČUJE DC-COMPENSATION kolo."
- moved on the sheet: C10, C21, C22, C23, C25, C3, C6, C8, R14, R15, R16, R17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
