File: power_supply.kicad_sch (KiCad schematic)
At the start: 62 parts, among them Q10 AO3401A, Q13 AO3400A, Q14 AO3400A, Q3 AO3400A, Q5 AO3400A, Q8 AO3401A, SW2 SW_DPDT_x2, U11 AP9101CK6, U6 BQ21040DBV, U7 74HC14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

Commit message: updated form factor and placment
Parts:
- removed D6: LED, LED_THT:LED_D3.0mm_FlatTop, symbol Device:LED
- added D3: GREEN_LED, LED_SMD:LED_0805_2012Metric_Pad1.15x1.40mm_HandSolder, symbol Device:LED
- added D5: RED_LED, LED_SMD:LED_0805_2012Metric_Pad1.15x1.40mm_HandSolder, symbol Device:LED
- R25: Type (none) -> NTC
- SW2: footprint DS100M08KV:DPDT_bigger -> PEKG:SW_EG1271
Connections:
- net at U6.3 (~{CHG}): now also D5.1 (K)
- net at R5.1: now also D5.2 (A)
Other:
- moved on the sheet: BT2, C6, Q3, Q5, R30, R8, U11

Commit message: ADC, levels
Parts:
- added R1: 1k, Resistor_SMD:R_0603_1608Metric_Pad0.98x0.95mm_HandSolder, symbol Device:R
- U7: footprint (none) -> Package_SO:SOIC-14_3.9x8.7mm_P1.27mm
- U7: renamed from U8; footprint (none) -> Package_SO:SOIC-14_3.9x8.7mm_P1.27mm
Connections:
- net +VIN: now also R1.2
- net GND: now also D3.1 (K)
- net at D3.2 (A): now also R1.1
Other:
- moved on the sheet: D3, SW2A, SW2B
