File: PEKG.kicad_pcb (KiCad board)
At the start: 2 copper layers, 90 x 45 mm, 132 parts, among them J1 AudioJack4, J2 EKG input, J3 Micro_SD_Card_Module, Q10 AO3401A, Q13 AO3400A, Q14 AO3400A, Q3 AO3400A, Q5 AO3400A, Q8 AO3401A, SW2 SW_DPDT_x2, U1 OP07, U11 AP9101CK6, U2 ESP32-S3-ZERO, U3 OP07, U4 NE5532, U5 NE5532, U6 BQ21040DBV, U7 74HC14

Commit message: charge pump placement
Parts:
- removed C111, C59: 100n, Capacitor_SMD:C_0603_1608Metric_Pad1.08x0.95mm_HandSolder
- removed C61, C62, C63, C64: 47u, Capacitor_THT:CP_Radial_D5.0mm_P2.00mm
- removed R19: 39k, Resistor_SMD:R_0603_1608Metric_Pad0.98x0.95mm_HandSolder
- removed R21, R39: 470k, Resistor_SMD:R_0603_1608Metric_Pad0.98x0.95mm_HandSolder
- added C10: 10u, Resistor_SMD:R_0805_2012Metric_Pad1.20x1.40mm_HandSolder, F.Cu at (164.7, 114.2)
- added C35: 100n, Capacitor_SMD:C_0603_1608Metric_Pad1.08x0.95mm_HandSolder, F.Cu at (150.4, 109.3)
- added C55: 10u, Resistor_SMD:R_0805_2012Metric_Pad1.20x1.40mm_HandSolder, F.Cu at (164.7, 112.3)
- added C56: 10u, Resistor_SMD:R_0805_2012Metric_Pad1.20x1.40mm_HandSolder, F.Cu at (164.7, 110.4)
- added C57: 10u, Resistor_SMD:R_0805_2012Metric_Pad1.20x1.40mm_HandSolder, F.Cu at (164.7, 108.5)
- added C58: 10u, Resistor_SMD:R_0805_2012Metric_Pad1.20x1.40mm_HandSolder, F.Cu at (164.7, 106.6)
- added JP5: Jumper_2_Open, Jumper:SolderJumper-2_P1.3mm_Open_RoundedPad1.0x1.5mm, F.Cu at (179.2, 107.1)
- added R51: 20k, Resistor_SMD:R_0603_1608Metric_Pad0.98x0.95mm_HandSolder, F.Cu at (176.2, 108.0)
- moved C1 268.9 mm to (150.2, 114.8)
- moved C41 265.9 mm to (157.5, 106.8), turned to 180 degrees
- moved C4 265.6 mm to (153.9, 118.9), turned to 180 degrees
- moved C2 261.6 mm to (157.5, 117.8), turned to 180 degrees
- moved C31 258.5 mm to (164.5, 115.9), turned to 180 degrees
- moved C5 252.4 mm to (169.0, 108.0)
- moved C42 235.2 mm to (153.9, 105.8)
- moved C17 202.2 mm to (173.4, 105.4), turned to -90 degrees
- moved Q14 111.8 mm to (153.9, 110.4), turned to -90 degrees
- moved Q10 110.2 mm to (153.9, 114.3), turned to 90 degrees
- moved D13 109.9 mm to (153.9, 107.5)
- moved C54 106.9 mm to (150.2, 111.0)
- moved C53 105.9 mm to (150.2, 112.9)
- moved C52 105.0 mm to (150.2, 116.7)
- moved C51 104.6 mm to (150.2, 118.6)
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Connections:
- D9 pad 2: CLK -> Net-(D9-A)
- R38 pad 2: CLK -> Net-(D9-A)
