File: mcu.kicad_sch (KiCad schematic)
At the start: 6 parts, among them J3 Micro_SD_Card_Module, U2 ESP32-S3-ZERO

Commit message: routing pending
Connections:
- no-connect marks 0 -> 10
Changed lines of the file:
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@@
 		(color 0 0 0 0)
+	)
+	(no_connect
+		(at 76.2 82.55)
+	)
+	(no_connect
+		(at 111.76 69.85)
+	)
+	(no_connect
+		(at 76.2 69.85)
+	)
+	(no_connect
+		(at 111.76 67.31)
+	)
+	(no_connect
+		(at 76.2 67.31)
+	)
+	(no_connect
+		(at 76.2 85.09)
+	)
+	(no_connect
+		(at 76.2 77.47)
+	)
+	(no_connect
+		(at 111.76 72.39)
+	)
+	(no_connect
+		(at 76.2 80.01)
+	)
+	(no_connect
+		(at 111.76 74.93)
 	)
 	(wire

Commit message: 99% done
Connections:
- net GND renamed 0
Changed lines of the file:
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@@
 			)
 		)
-		(property "Value" "GND"
+		(property "Value" "0"
 			(at 161.29 87.63 0)
 			(hide yes)
@@
 			)
 		)
-		(property "Value" "GND"
+		(property "Value" "0"
 			(at 60.96 97.79 0)
 			(hide yes)
@@
 			)
 		)
-		(property "Value" "GND"
+		(property "Value" "0"
 			(at 113.03 96.52 0)
 			(hide yes)
