File: amplifier.kicad_sch (KiCad schematic)
At the start: 57 parts, among them J2 EKG input, U1 OP07, U3 OP07, U4 NE5532, U5 NE5532

Commit message: rest placed
Parts:
- added C29: 10u, Capacitor_SMD:C_0603_1608Metric_Pad1.08x0.95mm_HandSolder, symbol Device:C
- added C45: 100n, Capacitor_SMD:C_0603_1608Metric_Pad1.08x0.95mm_HandSolder, symbol Device:C
- D1, D2: LCSC (none) -> C2500
Connections:
- net V_{ref} is gone; now on net GND: R26.1, U5.5 (+)
- net GND: no longer D1.1 (K), D2.1 (K)
- net V_{cc}: now also C29.1, C45.2
- net V_{ee}: now also D1.1 (K), D2.1 (K), C29.2, C45.1
Other:
- moved on the sheet: C26, C44, D1, TP13, U5C

Commit message: routing pending
Connections:
- no-connect marks 2 -> 6
Changed lines of the file:
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@@
+	)
+	(no_connect
+		(at 72.39 73.66)
+	)
+	(no_connect
+		(at 69.85 73.66)
+	)
+	(no_connect
+		(at 72.39 50.8)
 	)
 	(no_connect
 		(at 30.48 68.58)
 	)
+	(no_connect
+		(at 69.85 50.8)
+	)
 	(wire

Commit message: 99% done
Connections:
- net GND renamed 0

Commit message: basics done
Connections:
- net 3V3 is gone; now on net +3V3: R2.1
Changed lines of the file:
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@@
 		(in_pos_files yes)
 		(dnp no)
-		(fields_autoplaced yes)
 		(property "Reference" "#PWR019"
 			(at 209.55 80.01 0)
@@
 			)
 		)
-		(property "Value" "3V3"
-			(at 209.55 71.12 0)
+		(property "Value" "+3V3"
+			(at 207.01 71.12 0)
 			(show_name no)
 			(do_not_autoplace no)
@@
 					(size 1.27 1.27)
 				)
+				(justify left)
 			)
 		)
